File: KiCad/Gate reed.kicad_sch (KiCad schematic)
At the start: 0 parts

Commit message: Added comments  to the code and added mosfet to kicad scheme
Parts:
- added BT1: 18650 INR18650-35E 3450mAh 8A Li-ion, Battery:BatteryHolder_Keystone_1042_1x18650, symbol Device:Battery_Cell
- added C1, C2, C4: 0.1, symbol Device:C
- added C3, C6: 100u 16V, symbol Device:C_Polarized
- added C5: 100n 16V, symbol Device:C_Polarized
- added D1: Green LED, LED_THT:LED_D3.0mm, symbol Device:LED
- added J1, J2: Conn_01x02, Connector_JST:JST_XH_B2B-XH-A_1x02_P2.50mm_Vertical, symbol Connector_Generic:Conn_01x02
- added Q1: Q_PMOS_GSD, symbol Transistor_FET:Q_PMOS_GSD
- added R1: 470, Resistor_THT:R_Axial_DIN0207_L6.3mm_D2.5mm_P7.62mm_Horizontal, symbol Device:R
- added R2: 100k, Resistor_THT:R_Axial_DIN0207_L6.3mm_D2.5mm_P7.62mm_Horizontal, symbol Device:R
- added R3, R4, R6, R7: 220k, Resistor_THT:R_Axial_DIN0207_L6.3mm_D2.5mm_P7.62mm_Horizontal, symbol Device:R
- added R5: 100, Resistor_THT:R_Axial_DIN0207_L6.3mm_D2.5mm_P7.62mm_Horizontal, symbol Device:R
- added SW1: MTS-101 2-pin ON-OFF toggle switch, TerminalBlock_Phoenix:TerminalBlock_Phoenix_MKDS-1,5-2_1x02_P5.00mm_Horizontal, symbol Switch:SW_SPST
- added SW2: SW_Reed, Connector_JST:JST_XH_B2B-XH-A_1x02_P2.50mm_Vertical, symbol Switch:SW_Reed
- added U2: XIAO ESP32C3, XIAO_ESP32C3:xiao_esp32c3, symbol Xiao ESP32-C3:XIAO ESP32C3
Connections:
- new net: C5.1, C6.1, R4.1, SW1.2 (B), U2.B+ (Batt+)
- new net: C2.1, R3.1, R4.2, U2.1 (D0)
- new net: BT1.1 (+), J1.1 (Pin_1), Q1.2 (S), R7.1
- new net: Q1.1 (G), R6.1, R7.2
- new net: BT1.2 (-), C5.2, C6.2, J1.2 (Pin_2), R6.2, U2.B- (Batt-)
- new net: Q1.3 (D), SW1.1 (A)
- new net: J2.1 (Pin_1), R5.1, SW2.2
- new net: D1.2 (A), R1.2
- new net: C1.1, R2.2, R5.2, U2.3 (D2)
- new net: D1.1 (K), U2.8 (D7)
- new net +3.3V: C3.1, C4.1, R1.1, R2.1, U2.12 (VCC_3V3)
- new net GND: C1.2, C2.2, C3.2, C4.2, J2.2 (Pin_2), R3.2, SW2.1, U2.13 (GND)
- no-connect marks 0 -> 9
Other:
- company: (none) -> DIY
- title: (none) -> Gate Reed Monitor
